Commit message: base and realsense urdf.xacro added

File: xacro/robotont_base.urdf.xacro (robot description, xacro)
@@ -4,5 +4,4 @@
     <xacro:property name= "prefix" value="$(arg prefix)"/>
     <xacro:include filename="$(find robotont_description)/xacro/rim.urdf.xacro"/>
-    <xacro:include filename="$(find robotont_description)/xacro/_d435.urdf.xacro"/>
     <xacro:property name="wheel_distance" value="0.146" />
     <xacro:property name="wheel_center_height" value="0.021" />
@@ -47,34 +46,7 @@
 		/>
     </joint>
-    <!-- Camera -->
-    <!-- <link name="right_camera_boom"><visual><geometry><box size="0.005 0.16 0.01"/></geometry><origin rpy="0 0 0" xyz="0 0 0"/><material name="boom_material"><color rgba="1 1 1 0.7"/></material></visual><collision><geometry><box size="0.005 0.16 0.01"/></geometry><origin rpy="0 0 0" xyz="0 0 0"/></collision></link><joint
-		name="right_camera_boom_joint"
-		type="fixed"
-	><parent link="base_link" /><child link="right_camera_boom" /><origin
-			xyz="-0.05 0.145 -0.1"
-			rpy="0 0 0"
-		/></joint><link name="left_camera_boom"><visual><geometry><box size="0.005 0.16 0.01"/></geometry><origin rpy="0 0 0" xyz="0 0 0"/><material name="boom_material"><color rgba="1 1 1 0.7"/></material></visual><collision><geometry><box size="0.005 0.16 0.01"/></geometry><origin rpy="0 0 0" xyz="0 0 0"/></collision></link><joint
-		name="left_camera_boom_joint"
-		type="fixed"
-	><parent link="base_link" /><child link="left_camera_boom" /><origin
-			xyz="0.05 0.145 -0.1"
-			rpy="0 0 0"
-		/></joint><link name="camera_base"><visual><geometry><box size="0.1 0.02 0.005"/></geometry><origin rpy="0 0 0" xyz="0 0 0"/><material name="boom_material"><color rgba="1 1 1 0.7"/></material></visual></link><joint
-		name="camera_boom_to_base_joint"
-		type="fixed"
-	><parent link="right_camera_boom" /><child link="camera_base" /><origin
-			xyz="0.0475 0.07 0"
-			rpy="0 0 0"
-		/></joint> -->
     <sensor_d435 parent="${prefix}base_link" prefix="${prefix}">
         <origin xyz="-0.12 0 0.21" rpy="0 0 0"/>
     </sensor_d435>
-    <!-- <link name="camera_link"><origin rpy="0 0 0" xyz="0 0 0"/></link><joint
-		name="camera_base_to_link_joint"
-		type="fixed"
-	><parent link="camera_base" /><child link="camera_link" /><origin
-			xyz="0 0 0.011"
-			rpy="0 0 0"
-		/></joint> -->
     <!-- Computer -->
     <link name="${prefix}computer_link">
