Commit message: two launch files + simplebody.stl turned 90 deg

File: urdf/robotont_base.urdf.xacro (robot description, xacro)
@@ -32,5 +32,5 @@
                 <mesh scale=" 0.001 0.001 0.001" filename="package://robotont_description/meshes/simplebody.stl"/>
             </geometry>
-            <origin rpy="${pi/2} 0 0"  xyz="0 0 0"/>
+            <origin rpy="${pi/2} 0 ${pi/2}"  xyz="0 0 0"/>
         </collision>
     </link>
