Commit message: removed computer_link and gazebo from xacro files

File: urdf/rim.urdf.xacro (robot description, xacro)
@@ -176,8 +176,4 @@
 		/>
         <!-- <transmission name="rim_${name}_transmission"><type>transmission_interface/SimpleTransmission</type><joint name="rim_${name}_joint"><hardwareInterface>hardware_interface/EffortJointInterface</hardwareInterface></joint><actuator name="rim_${name}_motor"><mechanicalReduction>1</mechanicalReduction></actuator></transmission> -->
-        <gazebo reference="${prefix}rim_${name}_link">
-            <material>Gazebo/DarkGrey</material>
-            <!-- <kp>1000000</kp><kd>100</kd> -->
-        </gazebo>
     </xacro:macro>
 </robot>

File: urdf/robotont_base.urdf.xacro (robot description, xacro)
@@ -46,30 +46,4 @@
 		/>
     </joint>
-    <sensor_d435 parent="${prefix}base_link" prefix="${prefix}">
-        <origin xyz="-0.12 0 0.21" rpy="0 0 0"/>
-    </sensor_d435>
-    <!-- Computer -->
-    <link name="${prefix}computer_link">
-        <visual>
-            <geometry>
-                <box size="0.11 0.11 0.04"/>
-            </geometry>
-            <origin rpy="0 0 0" xyz="0 0 0"/>
-            <material name="computer_material">
-                <color rgba="0.1 0.1 0.1 1"/>
-            </material>
-        </visual>
-    </link>
-    <joint
-		name="${prefix}computer_joint"
-		type="fixed"
-	>
-        <parent link="${prefix}base_link" />
-        <child link="${prefix}computer_link" />
-        <origin
-			xyz="-0.01 0 0.085"
-			rpy="0 0 0"
-		/>
-    </joint>
     <!-- Wheels -->
     <xacro:rim_macro
@@ -97,62 +71,3 @@
         prefix="${prefix}"
 	/>
-    <!-- Initialize controller manager and odometry-->
-    <!-- libgazebo_ros_planar_move.so -->
-    <gazebo>
-        <plugin name="robotont_controller" filename="libgazebo_ros_planar_move.so">
-            <commandTopic>/robotont/cmd_vel</commandTopic>
-            <odometryTopic>/robotont/odom</odometryTopic>
-            <odometryFrame>odom</odometryFrame>
-            <odometryRate>30.0</odometryRate>
-            <robotBaseFrame>${prefix}base_footprint</robotBaseFrame>
-        </plugin>
-    </gazebo>
-    <!-- Give materials to links -->
-    <gazebo reference="${prefix}base_link">
-        <material>Robotont/BlueishTransparent</material>
-    </gazebo>
-    <gazebo reference="${prefix}camera_link">
-        <material>Gazebo/Grey</material>
-    </gazebo>
-    <gazebo reference="${prefix}computer_link">
-        <material>Gazebo/Black</material>
-    </gazebo>
-    <!-- Depth camera plugin -->
-    <gazebo reference="${prefix}camera_link">
-        <sensor type="depth" name="camera">
-            <always_on>true</always_on>
-            <update_rate>10.0</update_rate>
-            <camera>
-                <horizontal_fov>${90.0*pi/180.0}</horizontal_fov>
-                <image>
-                    <format>B8G8R8</format>
-                    <width>640</width>
-                    <height>480</height>
-                </image>
-                <clip>
-                    <near>0.02</near>
-                    <far>8.0</far>
-                </clip>
-            </camera>
-            <plugin name="kinect_camera_controller" filename="libgazebo_ros_openni_kinect.so">
-                <robotNamespace>/</robotNamespace>
-                <cameraName>camera</cameraName>
-                <alwaysOn>true</alwaysOn>
-                <updateRate>0.0</updateRate>
-                <imageTopicName>color/image_raw</imageTopicName>
-                <depthImageTopicName>depth/image_raw</depthImageTopicName>
-                <pointCloudTopicName>depth/points</pointCloudTopicName>
-                <cameraInfoTopicName>color/camera_info</cameraInfoTopicName>
-                <depthImageCameraInfoTopicName>depth/camera_info</depthImageCameraInfoTopicName>
-                <frameName>camera_depth_optical_frame</frameName>
-                <baseline>0.1</baseline>
-                <distortion_k1>0.0</distortion_k1>
-                <distortion_k2>0.0</distortion_k2>
-                <distortion_k3>0.0</distortion_k3>
-                <distortion_t1>0.0</distortion_t1>
-                <distortion_t2>0.0</distortion_t2>
-                <pointCloudCutoff>0.4</pointCloudCutoff>
-            </plugin>
-        </sensor>
-    </gazebo>
-</robot>
+ </robot>

File: urdf/roller.urdf.xacro (robot description, xacro)
@@ -44,7 +44,4 @@
 			/>
         </joint>
-        <gazebo reference="${prefix}roller_${name}_rim_${parent}_link">
-            <material>Robotont/DarkGreen</material>
-        </gazebo>
     </xacro:macro>
 </robot>

Commit message: corrected package.xml and readme, replaced tabs with spaces in rim.urdf.xacro

File: urdf/rim.urdf.xacro (robot description, xacro)
@@ -8,16 +8,16 @@
     <xacro:property name="roller_init_angle" value="0" />
     <xacro:macro name="rim_macro" params="name color angle wheel_distance wheel_center_height prefix">
-		<link name="${prefix}rim_${name}_link">
+        <link name="${prefix}rim_${name}_link">
             <inertial>
                 <origin xyz="0 0 0"/>
                 <mass value="0.00835758"/>
                 <inertia
-					ixx="6.63684e-07"
-					ixy="0"
-					ixz="0"
-					iyy="6.63684e-07"
-					iyz="0"
-					izz="9.40333e-07"
-				/>
+                    ixx="6.63684e-07"
+                    ixy="0"
+                    ixz="0"
+                    iyy="6.63684e-07"
+                    iyz="0"
+                    izz="9.40333e-07"
+                />
             </inertial>
             <visual>
@@ -36,143 +36,143 @@
         </link>
         <joint
-			name="${prefix}rim_${name}_joint"
-			type="continuous"
-		>
+            name="${prefix}rim_${name}_joint"
+            type="continuous"
+        >
             <parent link="${prefix}base_link" />
             <child link="${prefix}rim_${name}_link" />
             <axis xyz="0 0 1"/>
             <origin
-				xyz="${wheel_distance*sin(angle)} ${-wheel_distance*cos(angle)} ${wheel_center_height}"
-				rpy="${pi/2} 0 ${angle+pi}"
-			/>
+                xyz="${wheel_distance*sin(angle)} ${-wheel_distance*cos(angle)} ${wheel_center_height}"
+                rpy="${pi/2} 0 ${angle+pi}"
+            />
         </joint>
         <!-- Front rollers -->
         <xacro:roller_macro
-			parent="${name}"
-			radial_dist="${roller_radial_dist}"
-			z_distance="${roller_z_distance}"
-			z_distance_reflect="-1"
-			init_angle="${roller_init_angle}"
-			no_of_roller="0"
-			prefix="${prefix}"
-		/>
+            parent="${name}"
+            radial_dist="${roller_radial_dist}"
+            z_distance="${roller_z_distance}"
+            z_distance_reflect="-1"
+            init_angle="${roller_init_angle}"
+            no_of_roller="0"
+            prefix="${prefix}"
+        />
         <xacro:roller_macro
-			parent="${name}"
-			radial_dist="${roller_radial_dist}"
-			z_distance="${roller_z_distance}"
-			z_distance_reflect="-1"
-			init_angle="${roller_init_angle}"
-			no_of_roller="1"
-			prefix="${prefix}"
-		/>
+            parent="${name}"
+            radial_dist="${roller_radial_dist}"
+            z_distance="${roller_z_distance}"
+            z_distance_reflect="-1"
+            init_angle="${roller_init_angle}"
+            no_of_roller="1"
+            prefix="${prefix}"
+        />
         <xacro:roller_macro
-			parent="${name}"
-			radial_dist="${roller_radial_dist}"
-			z_distance="${roller_z_distance}"
-			z_distance_reflect="-1"
-			init_angle="${roller_init_angle}"
-			no_of_roller="2"
-			prefix="${prefix}"
-		/>
+            parent="${name}"
+            radial_dist="${roller_radial_dist}"
+            z_distance="${roller_z_distance}"
+            z_distance_reflect="-1"
+            init_angle="${roller_init_angle}"
+            no_of_roller="2"
+            prefix="${prefix}"
+        />
         <xacro:roller_macro
-			parent="${name}"
-			radial_dist="${roller_radial_dist}"
-			z_distance="${roller_z_distance}"
-			z_distance_reflect="-1"
-			init_angle="${roller_init_angle}"
-			no_of_roller="3"
-			prefix="${prefix}"
-		/>
+            parent="${name}"
+            radial_dist="${roller_radial_dist}"
+            z_distance="${roller_z_distance}"
+            z_distance_reflect="-1"
+            init_angle="${roller_init_angle}"
+            no_of_roller="3"
+            prefix="${prefix}"
+        />
         <xacro:roller_macro
-			parent="${name}"
-			radial_dist="${roller_radial_dist}"
-			z_distance="${roller_z_distance}"
-			z_distance_reflect="-1"
-			init_angle="${roller_init_angle}"
-			no_of_roller="4"
-			prefix="${prefix}"
-		/>
+            parent="${name}"
+            radial_dist="${roller_radial_dist}"
+            z_distance="${roller_z_distance}"
+            z_distance_reflect="-1"
+            init_angle="${roller_init_angle}"
+            no_of_roller="4"
+            prefix="${prefix}"
+        />
         <xacro:roller_macro
-			parent="${name}"
-			radial_dist="${roller_radial_dist}"
-			z_distance="${roller_z_distance}"
-			z_distance_reflect="-1"
-			init_angle="${roller_init_angle}"
-			no_of_roller="5"
-			prefix="${prefix}"
-		/>
+            parent="${name}"
+            radial_dist="${roller_radial_dist}"
+            z_distance="${roller_z_distance}"
+            z_distance_reflect="-1"
+            init_angle="${roller_init_angle}"
+            no_of_roller="5"
+            prefix="${prefix}"
+        />
         <xacro:roller_macro
-			parent="${name}"
-			radial_dist="${roller_radial_dist}"
-			z_distance="${roller_z_distance}"
-			z_distance_reflect="-1"
-			init_angle="${roller_init_angle}"
-			no_of_roller="6"
-			prefix="${prefix}"
-		/>
+            parent="${name}"
+            radial_dist="${roller_radial_dist}"
+            z_distance="${roller_z_distance}"
+            z_distance_reflect="-1"
+            init_angle="${roller_init_angle}"
+            no_of_roller="6"
+            prefix="${prefix}"
+        />
         <!-- Back rollers -->
         <xacro:roller_macro
-			parent="${name}"
-			radial_dist="${roller_radial_dist}"
-			z_distance="${roller_z_distance}"
-			z_distance_reflect="1"
-			init_angle="${roller_init_angle}"
-			no_of_roller="0"
-			prefix="${prefix}"
-		/>
+            parent="${name}"
+            radial_dist="${roller_radial_dist}"
+            z_distance="${roller_z_distance}"
+            z_distance_reflect="1"
+            init_angle="${roller_init_angle}"
+            no_of_roller="0"
+            prefix="${prefix}"
+        />
         <xacro:roller_macro
-			parent="${name}"
-			radial_dist="${roller_radial_dist}"
-			z_distance="${roller_z_distance}"
-			z_distance_reflect="1"
-			init_angle="${roller_init_angle}"
-			no_of_roller="1"
-			prefix="${prefix}"
-		/>
+            parent="${name}"
+            radial_dist="${roller_radial_dist}"
+            z_distance="${roller_z_distance}"
+            z_distance_reflect="1"
+            init_angle="${roller_init_angle}"
+            no_of_roller="1"
+            prefix="${prefix}"
+        />
         <xacro:roller_macro
-			parent="${name}"
-			radial_dist="${roller_radial_dist}"
-			z_distance="${roller_z_distance}"
-			z_distance_reflect="1"
-			init_angle="${roller_init_angle}"
-			no_of_roller="2"
-			prefix="${prefix}"
-		/>
+            parent="${name}"
+            radial_dist="${roller_radial_dist}"
+            z_distance="${roller_z_distance}"
+            z_distance_reflect="1"
+            init_angle="${roller_init_angle}"
+            no_of_roller="2"
+            prefix="${prefix}"
+        />
         <xacro:roller_macro
-			parent="${name}"
-			radial_dist="${roller_radial_dist}"
-			z_distance="${roller_z_distance}"
-			z_distance_reflect="1"
-			init_angle="${roller_init_angle}"
-			no_of_roller="3"
-			prefix="${prefix}"
-		/>
+            parent="${name}"
+            radial_dist="${roller_radial_dist}"
+            z_distance="${roller_z_distance}"
+            z_distance_reflect="1"
+            init_angle="${roller_init_angle}"
+            no_of_roller="3"
+            prefix="${prefix}"
+        />
         <xacro:roller_macro
-			parent="${name}"
-			radial_dist="${roller_radial_dist}"
-			z_distance="${roller_z_distance}"
-			z_distance_reflect="1"
-			init_angle="${roller_init_angle}"
-			no_of_roller="4"
-			prefix="${prefix}"
-		/>
+            parent="${name}"
+            radial_dist="${roller_radial_dist}"
+            z_distance="${roller_z_distance}"
+            z_distance_reflect="1"
+            init_angle="${roller_init_angle}"
+            no_of_roller="4"
+            prefix="${prefix}"
+        />
         <xacro:roller_macro
-			parent="${name}"
-			radial_dist="${roller_radial_dist}"
-			z_distance="${roller_z_distance}"
-			z_distance_reflect="1"
-			init_angle="${roller_init_angle}"
-			no_of_roller="5"
-			prefix="${prefix}"
-		/>
+            parent="${name}"
+            radial_dist="${roller_radial_dist}"
+            z_distance="${roller_z_distance}"
+            z_distance_reflect="1"
+            init_angle="${roller_init_angle}"
+            no_of_roller="5"
+            prefix="${prefix}"
+        />
         <xacro:roller_macro
-			parent="${name}"
-			radial_dist="${roller_radial_dist}"
-			z_distance="${roller_z_distance}"
-			z_distance_reflect="1"
-			init_angle="${roller_init_angle}"
-			no_of_roller="6"
-			prefix="${prefix}"
-		/>
+            parent="${name}"
+            radial_dist="${roller_radial_dist}"
+            z_distance="${roller_z_distance}"
+            z_distance_reflect="1"
+            init_angle="${roller_init_angle}"
+            no_of_roller="6"
+            prefix="${prefix}"
+        />
         <!-- <transmission name="rim_${name}_transmission"><type>transmission_interface/SimpleTransmission</type><joint name="rim_${name}_joint"><hardwareInterface>hardware_interface/EffortJointInterface</hardwareInterface></joint><actuator name="rim_${name}_motor"><mechanicalReduction>1</mechanicalReduction></actuator></transmission> -->
     </xacro:macro>

Commit message: cleaned up the style in xacro files, no functional changes

File: urdf/rim.urdf.xacro (robot description, xacro)
@@ -9,16 +9,4 @@
     <xacro:macro name="rim_macro" params="name color angle wheel_distance wheel_center_height prefix">
         <link name="${prefix}rim_${name}_link">
-            <inertial>
-                <origin xyz="0 0 0"/>
-                <mass value="0.00835758"/>
-                <inertia
-                    ixx="6.63684e-07"
-                    ixy="0"
-                    ixz="0"
-                    iyy="6.63684e-07"
-                    iyz="0"
-                    izz="9.40333e-07"
-                />
-            </inertial>
             <visual>
                 <geometry>
@@ -34,9 +22,18 @@
                 </geometry>
             </collision>
+            <inertial>
+                <origin xyz="0 0 0"/>
+                <mass value="0.00835758"/>
+                <inertia
+                    ixx="6.63684e-07"
+                    ixy="0"
+                    ixz="0"
+                    iyy="6.63684e-07"
+                    iyz="0"
+                    izz="9.40333e-07"
+                />
+            </inertial>
         </link>
-        <joint
-            name="${prefix}rim_${name}_joint"
-            type="continuous"
-        >
+        <joint name="${prefix}rim_${name}_joint" type="continuous">
             <parent link="${prefix}base_link" />
             <child link="${prefix}rim_${name}_link" />

File: urdf/robotont_base.urdf.xacro (robot description, xacro)
@@ -4,19 +4,8 @@
     <xacro:property name= "prefix" value="$(arg prefix)"/>
     <xacro:include filename="$(find robotont_description)/urdf/rim.urdf.xacro"/>
-    <xacro:property name="wheel_distance" value="0.146" />
-    <xacro:property name="wheel_center_height" value="0.021" />
+    <xacro:property name="wheel_distance" value="0.146"/>
+    <xacro:property name="wheel_center_height" value="0.021"/>
     <link name="${prefix}base_footprint"/>
     <link name="${prefix}base_link">
-        <inertial>
-            <mass value="3"/>
-            <inertia
-			ixx="0.00002035985530754"
-			ixy="0"
-			ixz="0"
-			iyy="0.00002035985530754"
-			iyz="0"
-			izz="0.00003945961663220"
-		/>
-        </inertial>
         <visual>
             <geometry>
@@ -30,19 +19,24 @@
         <collision>
             <geometry>
-                <mesh scale=" 0.001 0.001 0.001" filename="package://robotont_description/meshes/simplebody.stl"/>
+                <mesh scale="0.001 0.001 0.001" filename="package://robotont_description/meshes/simplebody.stl"/>
             </geometry>
             <origin rpy="${pi/2} 0 ${pi/2}"  xyz="0 0 0"/>
         </collision>
+        <inertial>
+            <mass value="3"/>
+            <inertia
+			    ixx="0.00002035985530754"
+			    ixy="0"
+			    ixz="0"
+			    iyy="0.00002035985530754"
+			    iyz="0"
+			    izz="0.00003945961663220"
+		    />
+        </inertial>
     </link>
-    <joint
-		name="${prefix}base_joint"
-		type="fixed"
-	>
-        <parent link="${prefix}base_footprint" />
-        <child link="${prefix}base_link" />
-        <origin
-			xyz="0 0 0.013"
-			rpy="0 0 0"
-		/>
+    <joint name="${prefix}base_joint" type="fixed">
+        <parent link="${prefix}base_footprint"/>
+        <child link="${prefix}base_link"/>
+        <origin xyz="0 0 0.013" rpy="0 0 0"/>
     </joint>
     <!-- Wheels -->

File: urdf/roller.urdf.xacro (robot description, xacro)
@@ -15,4 +15,12 @@
         </xacro:unless>
         <link name="${prefix}roller_${name}_rim_${parent}_link">
+            <visual>
+                <geometry>
+                    <mesh scale="0.001 0.001 0.001" filename="package://robotont_description/meshes/roller.stl"/>
+                </geometry>
+                <material name="roller_material">
+                    <color rgba="0.1 1 0.3 1"/>
+                </material>
+            </visual>
             <!-- <inertial><mass value="0.00113845"/><inertia
 					ixx="2.53776e-08"
@@ -23,12 +31,4 @@
 					izz="1.47666e-08"
 				/></inertial> -->
-            <visual>
-                <geometry>
-                    <mesh scale="0.001 0.001 0.001" filename="package://robotont_description/meshes/roller.stl"/>
-                </geometry>
-                <material name="roller_material">
-                    <color rgba="0.1 1 0.3 1"/>
-                </material>
-            </visual>
         </link>
         <joint
