Commit message: - Add description for robotont gen3 - Add launch parameter to switch between gen2.1 and 3 descriptions - Update package structure and xacro files

File: urdf/shared/rim.urdf.xacro (robot description, xacro)
@@ -2,17 +2,17 @@
 <robot
     xmlns:xacro="http://ros.org/wiki/xacro">
-    <xacro:include filename="$(find robotont_description)/urdf/roller.urdf.xacro"/>
-    <!-- Roller positioning -->
+    <xacro:include filename="$(find robotont_description)/urdf/shared/roller.urdf.xacro"/>
     <xacro:property name="roller_radial_dist" value="0.0275" />
     <xacro:property name="roller_z_distance" value="0.008" />
     <xacro:property name="roller_init_angle" value="0" />
-    <xacro:macro name="rim_macro" params="name color angle wheel_distance wheel_center_height prefix">
+    <xacro:property name="wheel_height_offset" value="${wheel_center_height / 2}"/>
+    <xacro:macro name="rim_macro" params="name color roller_color angle wheel_distance wheel_center_height z_rotation_offset prefix">
         <link name="${prefix}rim_${name}_link">
             <visual>
                 <geometry>
-                    <mesh filename="package://robotont_description/meshes/rim.stl"/>
+                    <mesh filename="package://robotont_description/meshes/shared/rim.STL"/>
                 </geometry>
                 <material name="rim_${name}_material">
-                    <color rgba="${color} 1"/>
+                    <color rgba="${color}"/>
                 </material>
             </visual>
@@ -23,5 +23,5 @@
             </collision>
             <inertial>
-                <origin xyz="0 0 0"/>
+                <origin xyz="0 ${wheel_height_offset} 0"/>
                 <mass value="0.00835758"/>
                 <inertia
@@ -40,6 +40,6 @@
             <axis xyz="0 0 1"/>
             <origin
-                xyz="${wheel_distance*sin(angle)} ${-wheel_distance*cos(angle)} ${wheel_center_height}"
-                rpy="${pi/2} 0 ${angle+pi}"
+                xyz="${wheel_distance * sin(angle)} ${ -wheel_distance * cos(angle)} ${wheel_center_height + wheel_height_offset}"
+                rpy="${pi/2} 0 ${angle + pi + z_rotation_offset}"
             />
         </joint>
@@ -47,4 +47,5 @@
         <xacro:roller_macro
             parent="${name}"
+            color="${roller_color}"
             radial_dist="${roller_radial_dist}"
             z_distance="${roller_z_distance}"
@@ -56,4 +57,5 @@
         <xacro:roller_macro
             parent="${name}"
+            color="${roller_color}"
             radial_dist="${roller_radial_dist}"
             z_distance="${roller_z_distance}"
@@ -65,4 +67,5 @@
         <xacro:roller_macro
             parent="${name}"
+            color="${roller_color}"
             radial_dist="${roller_radial_dist}"
             z_distance="${roller_z_distance}"
@@ -74,4 +77,5 @@
         <xacro:roller_macro
             parent="${name}"
+            color="${roller_color}"
             radial_dist="${roller_radial_dist}"
             z_distance="${roller_z_distance}"
@@ -83,4 +87,5 @@
         <xacro:roller_macro
             parent="${name}"
+            color="${roller_color}"
             radial_dist="${roller_radial_dist}"
             z_distance="${roller_z_distance}"
@@ -92,4 +97,5 @@
         <xacro:roller_macro
             parent="${name}"
+            color="${roller_color}"
             radial_dist="${roller_radial_dist}"
             z_distance="${roller_z_distance}"
@@ -101,4 +107,5 @@
         <xacro:roller_macro
             parent="${name}"
+            color="${roller_color}"
             radial_dist="${roller_radial_dist}"
             z_distance="${roller_z_distance}"
@@ -111,4 +118,5 @@
         <xacro:roller_macro
             parent="${name}"
+            color="${roller_color}"
             radial_dist="${roller_radial_dist}"
             z_distance="${roller_z_distance}"
@@ -120,4 +128,5 @@
         <xacro:roller_macro
             parent="${name}"
+            color="${roller_color}"
             radial_dist="${roller_radial_dist}"
             z_distance="${roller_z_distance}"
@@ -129,4 +138,5 @@
         <xacro:roller_macro
             parent="${name}"
+            color="${roller_color}"
             radial_dist="${roller_radial_dist}"
             z_distance="${roller_z_distance}"
@@ -138,4 +148,5 @@
         <xacro:roller_macro
             parent="${name}"
+            color="${roller_color}"
             radial_dist="${roller_radial_dist}"
             z_distance="${roller_z_distance}"
@@ -147,4 +158,5 @@
         <xacro:roller_macro
             parent="${name}"
+            color="${roller_color}"
             radial_dist="${roller_radial_dist}"
             z_distance="${roller_z_distance}"
@@ -156,4 +168,5 @@
         <xacro:roller_macro
             parent="${name}"
+            color="${roller_color}"
             radial_dist="${roller_radial_dist}"
             z_distance="${roller_z_distance}"
@@ -165,4 +178,5 @@
         <xacro:roller_macro
             parent="${name}"
+            color="${roller_color}"
             radial_dist="${roller_radial_dist}"
             z_distance="${roller_z_distance}"
@@ -172,5 +186,4 @@
             prefix="${prefix}"
         />
-        <!-- <transmission name="rim_${name}_transmission"><type>transmission_interface/SimpleTransmission</type><joint name="rim_${name}_joint"><hardwareInterface>hardware_interface/EffortJointInterface</hardwareInterface></joint><actuator name="rim_${name}_motor"><mechanicalReduction>1</mechanicalReduction></actuator></transmission> -->
     </xacro:macro>
 </robot>

File: urdf/shared/roller.urdf.xacro (robot description, xacro)
@@ -4,5 +4,5 @@
     <xacro:macro
 		name="roller_macro"
-		params="parent radial_dist z_distance z_distance_reflect init_angle no_of_roller prefix"
+		params="parent color radial_dist z_distance z_distance_reflect init_angle no_of_roller prefix"
 	>
         <xacro:if value="${z_distance_reflect==-1}">
@@ -17,8 +17,8 @@
             <visual>
                 <geometry>
-                    <mesh scale="0.001 0.001 0.001" filename="package://robotont_description/meshes/roller.stl"/>
+                    <mesh scale="0.001 0.001 0.001" filename="package://robotont_description/meshes/shared/roller.STL"/>
                 </geometry>
                 <material name="roller_material">
-                    <color rgba="0.1 1 0.3 1"/>
+                    <color rgba="${color}"/>
                 </material>
             </visual>
@@ -32,11 +32,7 @@
 				/></inertial> -->
         </link>
-        <joint
-			name="${prefix}roller_${name}_rim_${parent}_joint"
-			type="fixed"
-		>
+        <joint name="${prefix}roller_${name}_rim_${parent}_joint" type="fixed">
             <parent link="${prefix}rim_${parent}_link"/>
             <child link="${prefix}roller_${name}_rim_${parent}_link"/>
-            <!-- <axis xyz="1 0 0"/> -->
             <origin
 				xyz="${radial_dist*sin(-1*z_distance_reflect*(init_angle+offset+no_of_roller*2*pi/7))} ${-radial_dist*cos(-1*z_distance_reflect*(init_angle+offset+no_of_roller*2*pi/7))} ${z_distance*z_distance_reflect}"
