Commit message: robotont-description - Separate motor from the bracket, set bracket color to match frame - Add more concise examples of usage to readme

File: urdf/gen2_1/motor.urdf.xacro (robot description, xacro)
@@ -3,20 +3,32 @@
     xmlns:xacro="http://ros.org/wiki/xacro">
     <xacro:property name="length" value="0.0946"/>
-    <xacro:macro name="motor_macro" params="name color angle wheel_center_height frame_ground_clearance frame_thickness distance gap z_rotation prefix">
+    <xacro:macro name="motor_macro" params="
+        name
+        color
+        motor_color
+        angle
+        wheel_center_height
+        frame_ground_clearance
+        frame_thickness
+        distance
+        gap
+        z_rotation
+        prefix
+    ">
         <xacro:property name="ground_clearance" value="${1.5 * wheel_center_height + frame_ground_clearance + frame_thickness}"/>
         <xacro:property name="distance_from_center" value="${distance + (wheel_center_height / 2) + (length / 2) + gap}"/>
-        <link name="${prefix}motor_${name}_link">
+        <link name="${prefix}motor_mount_${name}_link">
             <visual>
                 <geometry>
                     <mesh filename="package://robotont_description/meshes/gen2_1/motor_module.STL"/>
                 </geometry>
-                <material name="motor_${name}_material">
+                <material name="motor_mount_${name}_material">
                     <color rgba="${color}"/>
                 </material>
             </visual>
         </link>
-        <joint name="motor_${name}_joint" type="fixed">
+        <joint name="motor_mount_${name}_joint" type="fixed">
             <parent link="${prefix}base_link"/>
-            <child link="${prefix}motor_${name}_link"/>
+            <child link="${prefix}motor_mount_${name}_link"/>
             <axis xyz="0 0 1"/>
             <origin
@@ -25,4 +37,22 @@
             />
         </joint>
+        <link name="${prefix}motor_${name}_link">
+            <visual>
+                <geometry>
+                    <mesh filename="package://robotont_description/meshes/gen2_1/motor.STL"/>
+                </geometry>
+                <material name="motor_${name}_material">
+                    <color rgba="${motor_color}"/>
+                </material>
+            </visual>
+        </link>
+        <joint name="motor_${name}_joint" type="fixed">
+            <parent link="${prefix}motor_mount_${name}_link"/>
+            <child link="${prefix}motor_${name}_link"/>
+            <axis xyz="0 0 1"/>
+            <origin
+                xyz="0 -0.0028 -0.008"
+            />
+        </joint>
     </xacro:macro>
 </robot>

File: urdf/gen2_1/robotont.urdf.xacro (robot description, xacro)
@@ -11,4 +11,5 @@
     <xacro:property name="roller_color" value="0.45 0.7 0.5 1.0"/>
     <xacro:property name="rim_color" value="0.26 0.26 0.26 1.0"/>
+    <xacro:property name="motor_color" value="0.26 0.26 0.26 1.0"/>
     <xacro:property name="frame_height" value="0.065"/>
     <xacro:property name="frame_ground_clearance" value="0.01"/>
@@ -29,5 +30,6 @@
     <xacro:motor_macro
         name="back"
-        color="${rim_color}"
+        color="${base_color}"
+        motor_color="${motor_color}"
         angle="${-3 * pi/2}"
         z_rotation="0"
@@ -36,10 +38,11 @@
         frame_thickness="${frame_thickness}"
         distance="${-wheel_distance}"
-        gap="-0.008"
+        gap="-0.016"
         prefix="${prefix}"
     />
     <xacro:motor_macro
         name="right"
-        color="${rim_color}"
+        color="${base_color}"
+        motor_color="${motor_color}"
         angle="${5 * pi / 6}"
         z_rotation="${pi}"
@@ -48,10 +51,11 @@
         frame_thickness="${frame_thickness}"
         distance="${wheel_distance}"
-        gap="-0.108"
+        gap="-0.1"
         prefix="${prefix}"
     />
     <xacro:motor_macro
         name="left"
-        color="${rim_color}"
+        color="${base_color}"
+        motor_color="${motor_color}"
         angle="${7 * pi / 6}"
         z_rotation="0"
@@ -60,5 +64,5 @@
         frame_thickness="${frame_thickness}"
         distance="${-wheel_distance}"
-        gap="-0.008"
+        gap="-0.016"
         prefix="${prefix}"
     />
