Commit message: robotont-description - Update gen2.1 model

File: urdf/gen2_1/robotont.urdf.xacro (robot description, xacro)
@@ -75,5 +75,13 @@
         wheel_distance="${wheel_distance}"
         wheel_center_height="${wheel_center_height}"
-        z_rotation_offset="0"
+        prefix="${prefix}"
+    />
+    <xacro:rim_macro
+        name="left"
+        color="${rim_color}"
+        roller_color="${roller_color}"
+        angle="${5 * pi / 6}"
+        wheel_distance="${wheel_distance}"
+        wheel_center_height="${wheel_center_height}"
         prefix="${prefix}"
     />
@@ -82,18 +90,8 @@
         color="${rim_color}"
         roller_color="${roller_color}"
-        angle="${5 * pi / 6}"
-        wheel_distance="${wheel_distance}"
-        wheel_center_height="${wheel_center_height}"
-        z_rotation_offset="0"
-        prefix="${prefix}"
-    />
-    <xacro:rim_macro
-        name="left"
-        color="${rim_color}"
-        roller_color="${roller_color}"
         angle="${7 * pi / 6}"
+        flip_axis="-1"
         wheel_distance="${-wheel_distance}"
         wheel_center_height="${wheel_center_height}"
-        z_rotation_offset="0"
         prefix="${prefix}"
     />

File: urdf/gen3/robotont.urdf.xacro (robot description, xacro)
@@ -84,5 +84,5 @@
     />
     <xacro:rim_macro
-        name="right"
+        name="left"
         color="${rim_color}"
         roller_color="${roller_color}"
@@ -94,8 +94,9 @@
     />
     <xacro:rim_macro
-        name="left"
+        name="right"
         color="${rim_color}"
         roller_color="${roller_color}"
         angle="${7 * pi / 6}"
+        flip_axis="-1"
         wheel_distance="${-wheel_distance}"
         wheel_center_height="${wheel_center_height}"

File: urdf/shared/rim.urdf.xacro (robot description, xacro)
@@ -12,7 +12,8 @@
         roller_color
         angle
+        flip_axis:=1
         wheel_distance
         wheel_center_height
-        wheel_center_offset
+        wheel_center_offset:=0
         prefix
     ">
@@ -47,5 +48,5 @@
             <parent link="${prefix}base_link" />
             <child link="${prefix}rim_${name}_link" />
-            <axis xyz="0 0 1"/>
+            <axis xyz="0 0 ${flip_axis}"/>
             <origin
                 xyz="${wheel_center_offset + (wheel_distance * sin(angle))} ${ -wheel_distance * cos(angle)} ${wheel_center_height + wheel_height_offset}"
