Commit message: robotont-description - Update models, move camera + nuc to separate package - Update xacro file structure

File: urdf/gen2_1/base.urdf.xacro (robot description, xacro)
@@ -1,5 +1,13 @@
 <?xml version="1.0"?>
 <robot xmlns:xacro="http://ros.org/wiki/xacro">
-    <xacro:macro name="base_macro" params="color frame_height frame_ground_clearance prefix">
+    <xacro:property name="e_button_offset" value="0.0035"/>
+    <xacro:macro name="base_macro" params="
+        color
+        e_button_color
+        power_button_color
+        frame_height
+        frame_ground_clearance
+        prefix"
+    >
         <link name="${prefix}base_link">
             <visual>
@@ -35,4 +43,44 @@
             <origin xyz="0 0 ${frame_ground_clearance}" rpy="0 0 0"/>
         </joint>
+        <!-- E-button -->
+        <link name="${prefix}e_button_link">
+            <visual>
+                <geometry>
+                    <mesh filename="package://robotont_description/meshes/gen3/e_stop_button.STL"/>
+                </geometry>
+                <material name="e_button_material">
+                    <color rgba="${e_button_color}"/>
+                </material>
+            </visual>
+        </link>
+        <joint name="e_button_joint" type="fixed">
+            <parent link="${prefix}base_link"/>
+            <child link="${prefix}e_button_link"/>
+            <axis xyz="0 0 1"/>
+            <origin
+                xyz="-0.0094 0.105 ${frame_ground_clearance + frame_height - e_button_offset}"
+                rpy="${pi / 2} 0 ${pi / 2}"
+            />
+        </joint>
+        <!-- Power button -->
+        <link name="${prefix}power_button_link">
+            <visual>
+                <geometry>
+                    <mesh filename="package://robotont_description/meshes/gen3/power_button.STL"/>
+                </geometry>
+                <material name="power_button_material">
+                    <color rgba="${power_button_color}"/>
+                </material>
+            </visual>
+        </link>
+        <joint name="power_button_joint" type="fixed">
+            <parent link="${prefix}base_link"/>
+            <child link="${prefix}power_button_link"/>
+            <axis xyz="0 0 1"/>
+            <origin
+                xyz="-0.0094 0.133 ${frame_ground_clearance + frame_height - 0.001}"
+                rpy="${pi / 2} 0 ${pi / 2}"
+            />
+        </joint>
     </xacro:macro>
 </robot>

File: urdf/gen2_1/robotont.urdf.xacro (robot description, xacro)
@@ -3,18 +3,62 @@
     <xacro:include filename="$(find robotont_description)/urdf/shared/rim.urdf.xacro"/>
     <xacro:include filename="$(find robotont_description)/urdf/gen2_1/base.urdf.xacro"/>
+    <xacro:include filename="$(find robotont_description)/urdf/gen2_1/motor.urdf.xacro"/>
     <xacro:arg name="prefix" default=""/>
     <xacro:property name="prefix" value="$(arg prefix)"/>
     <xacro:property name="wheel_distance" value="0.146"/>
     <xacro:property name="wheel_center_height" value="0.021"/>
+    <xacro:property name="wheel_length" value="0.0225"/>
     <xacro:property name="roller_color" value="0.45 0.7 0.5 1.0"/>
     <xacro:property name="rim_color" value="0.26 0.26 0.26 1.0"/>
     <xacro:property name="frame_height" value="0.065"/>
-    <xacro:property name="frame_ground_clearance" value="0.014"/>
+    <xacro:property name="frame_ground_clearance" value="0.01"/>
+    <xacro:property name="frame_thickness" value="0.000025"/>
     <xacro:property name="base_color" value="1.0 1.0 1.0 0.6"/>
+    <xacro:property name="e_button_color" value="1.0 0 0 0.8"/>
+    <xacro:property name="power_button_color" value="0.75 0.75 0.75 1.0"/>
     <link name="${prefix}base_footprint"/>
     <xacro:base_macro
         color="${base_color}"
+        e_button_color="${e_button_color}"
+        power_button_color="${power_button_color}"
         frame_height="${frame_height}"
         frame_ground_clearance="${frame_ground_clearance}"
+        prefix="${prefix}"
+    />
+    <!-- Motor modules -->
+    <xacro:motor_macro
+        name="back"
+        color="${rim_color}"
+        angle="${-3 * pi/2}"
+        z_rotation="0"
+        wheel_center_height="${wheel_center_height}"
+        frame_ground_clearance="${frame_ground_clearance}"
+        frame_thickness="${frame_thickness}"
+        distance="${-wheel_distance}"
+        gap="-0.008"
+        prefix="${prefix}"
+    />
+    <xacro:motor_macro
+        name="right"
+        color="${rim_color}"
+        angle="${5 * pi / 6}"
+        z_rotation="${pi}"
+        wheel_center_height="${wheel_center_height}"
+        frame_ground_clearance="${frame_ground_clearance}"
+        frame_thickness="${frame_thickness}"
+        distance="${wheel_distance}"
+        gap="-0.108"
+        prefix="${prefix}"
+    />
+    <xacro:motor_macro
+        name="left"
+        color="${rim_color}"
+        angle="${7 * pi / 6}"
+        z_rotation="0"
+        wheel_center_height="${wheel_center_height}"
+        frame_ground_clearance="${frame_ground_clearance}"
+        frame_thickness="${frame_thickness}"
+        distance="${-wheel_distance}"
+        gap="-0.008"
         prefix="${prefix}"
     />
@@ -34,5 +78,5 @@
         color="${rim_color}"
         roller_color="${roller_color}"
-        angle="${-1/3*pi + pi/2}"
+        angle="${5 * pi / 6}"
         wheel_distance="${wheel_distance}"
         wheel_center_height="${wheel_center_height}"
@@ -44,6 +88,6 @@
         color="${rim_color}"
         roller_color="${roller_color}"
-        angle="${1/3*pi + pi/2}"
-        wheel_distance="${wheel_distance}"
+        angle="${7 * pi / 6}"
+        wheel_distance="${-wheel_distance}"
         wheel_center_height="${wheel_center_height}"
         z_rotation_offset="0"

File: urdf/gen3/base.urdf.xacro (robot description, xacro)
@@ -1,8 +1,21 @@
 <?xml version="1.0"?>
 <robot xmlns:xacro="http://ros.org/wiki/xacro">
-    <xacro:macro name="base_macro" params="color frame_height frame_ground_clearance prefix">
+    <xacro:property name="pcb_offset" value="0.044"/>
+    <xacro:property name="e_button_offset" value="0.0035"/>
+    <xacro:macro name="base_macro" params="
+        color
+        pcb_color
+        e_button_color
+        power_button_color
+        battery_module_color
+        frame_height
+        frame_ground_clearance
+        prefix
+    ">
+        <xacro:property name="frame_elevation" value="${frame_height / 2 + frame_ground_clearance}"/>
+        <!-- Frame -->
         <link name="${prefix}base_link">
             <visual>
-                <origin rpy="0 0 ${pi/2}" xyz="0 0 ${frame_height / 2 + frame_ground_clearance}"/>
+                <origin rpy="0 0 ${pi/2}" xyz="0 0 ${frame_elevation}"/>
                 <geometry>
                     <mesh filename="package://robotont_description/meshes/gen3/frame_module.STL"/>
@@ -16,5 +29,5 @@
                     <mesh filename="package://robotont_description/meshes/shared/collision_body.STL"/>
                 </geometry>
-                <origin rpy="${pi/2} 0 ${pi/2}" xyz="0 0 ${frame_height / 2 + frame_ground_clearance}"/>
+                <origin rpy="${pi/2} 0 ${pi/2}" xyz="0 0 ${frame_elevation}"/>
             </collision>
             <inertial>
@@ -33,5 +46,82 @@
             <parent link="${prefix}base_footprint"/>
             <child link="${prefix}base_link"/>
-            <origin xyz="0 0 0.013" rpy="0 0 0"/>
+            <origin xyz="0 0 ${frame_elevation}" rpy="0 0 0"/>
+        </joint>
+        <!-- PCB -->
+        <link name="${prefix}pcb_link">
+            <visual>
+                <origin rpy="0 0 ${pi/2}" xyz="0 0 0"/>
+                <geometry>
+                    <mesh filename="package://robotont_description/meshes/gen3/PCB.STL"/>
+                </geometry>
+                <material name="pcb_material">
+                    <color rgba="${pcb_color}"/>
+                </material>
+            </visual>
+        </link>
+        <joint name="${prefix}pcb_joint" type="fixed">
+            <parent link="${prefix}base_link"/>
+            <child link="${prefix}pcb_link"/>
+            <origin xyz="0.0025 0 ${frame_ground_clearance + pcb_offset}" rpy="0 ${pi / 2} 0"/>
+        </joint>
+        <!-- E-button -->
+        <link name="${prefix}e_button_link">
+            <visual>
+                <geometry>
+                    <mesh filename="package://robotont_description/meshes/gen3/e_stop_button.STL"/>
+                </geometry>
+                <material name="e_button_material">
+                    <color rgba="${e_button_color}"/>
+                </material>
+            </visual>
+        </link>
+        <joint name="e_button_joint" type="fixed">
+            <parent link="${prefix}base_link"/>
+            <child link="${prefix}e_button_link"/>
+            <axis xyz="0 0 1"/>
+            <origin
+                xyz="0.0075 0.115 ${frame_ground_clearance + frame_height - e_button_offset}"
+                rpy="${pi / 2} 0 ${pi / 2}"
+            />
+        </joint>
+        <!-- Power button -->
+        <link name="${prefix}power_button_link">
+            <visual>
+                <geometry>
+                    <mesh filename="package://robotont_description/meshes/gen3/power_button.STL"/>
+                </geometry>
+                <material name="power_button_material">
+                    <color rgba="${power_button_color}"/>
+                </material>
+            </visual>
+        </link>
+        <joint name="power_button_joint" type="fixed">
+            <parent link="${prefix}base_link"/>
+            <child link="${prefix}power_button_link"/>
+            <axis xyz="0 0 1"/>
+            <origin
+                xyz="-0.0472 0.111 ${frame_ground_clearance + frame_height - 0.001}"
+                rpy="${pi / 2} 0 ${pi / 2}"
+            />
+        </joint>
+        <!-- Battery module -->
+        <link name="${prefix}battery_module_link">
+            <visual>
+                <geometry>
+                    <mesh filename="package://robotont_description/meshes/gen3/battery_module.STL"/>
+                </geometry>
+                <material name="battery_module_material">
+                    <color rgba="${battery_module_color}"/>
+                </material>
+            </visual>
+        </link>
+        <joint name="battery_module_joint" type="fixed">
+            <parent link="${prefix}base_link"/>
+            <child link="${prefix}battery_module_link"/>
+            <axis xyz="0 0 1"/>
+            <origin
+                xyz="0.08 0 ${frame_ground_clearance + frame_height + 0.0025}"
+                rpy="${pi / 2} 0 ${pi / 2}"
+            />
         </joint>
     </xacro:macro>

File: urdf/gen3/robotont.urdf.xacro (robot description, xacro)
@@ -3,8 +3,5 @@
     <xacro:include filename="$(find robotont_description)/urdf/shared/rim.urdf.xacro"/>
     <xacro:include filename="$(find robotont_description)/urdf/gen3/motor.urdf.xacro"/>
-    <xacro:include filename="$(find robotont_description)/urdf/gen3/nuc.urdf.xacro"/>
-    <xacro:include filename="$(find robotont_description)/urdf/gen3/camera.urdf.xacro"/>
     <xacro:include filename="$(find robotont_description)/urdf/gen3/base.urdf.xacro"/>
-    <xacro:include filename="$(find robotont_description)/urdf/gen3/button.urdf.xacro"/>
     <xacro:arg name="prefix" default=""/>
     <xacro:property name="prefix" value="$(arg prefix)"/>
@@ -20,9 +17,16 @@
     <xacro:property name="frame_thickness" value="0.000025"/>
     <xacro:property name="base_color" value="0.16 0.65 0.98 1.0"/>
-    <xacro:property name="nuc_frame_color" value="0.75 0.75 0.75 1.0"/>
+    <xacro:property name="pcb_color" value="0 0.55 0.29 1.0"/>
+    <xacro:property name="e_button_color" value="1.0 0 0 0.8"/>
+    <xacro:property name="power_button_color" value="0.75 0.75 0.75 1.0"/>
+    <xacro:property name="battery_module_color" value="0.26 0.26 0.26 1.0"/>
     <link name="${prefix}base_footprint"/>
     <!-- Frame module -->
     <xacro:base_macro
         color="${base_color}"
+        pcb_color="${pcb_color}"
+        e_button_color="${e_button_color}"
+        power_button_color="${power_button_color}"
+        battery_module_color="${battery_module_color}"
         frame_height="${frame_height}"
         frame_ground_clearance="${frame_ground_clearance}"
@@ -100,24 +104,3 @@
         prefix="${prefix}"
     />
-    <!-- Computer module -->
-    <xacro:nuc_macro
-        color="${nuc_frame_color}"
-        frame_height="${frame_height}"
-        frame_ground_clearance="${frame_ground_clearance}"
-        prefix="${prefix}"
-    />
-    <!-- Camera module -->
-    <xacro:camera_macro
-        color="${nuc_frame_color}"
-        frame_height="${frame_height}"
-        frame_ground_clearance="${frame_ground_clearance}"
-        prefix="${prefix}"
-    />
-    <!-- E-button -->
-    <xacro:e_button_macro
-        color="1.0 0 0 1.0"
-        frame_height="${frame_height}"
-        frame_ground_clearance="${frame_ground_clearance}"
-        prefix="${prefix}"
-    />
 </robot>

Commit message: robotont-description - Make model compatible with gz sim 8

File: urdf/gen2_1/base.urdf.xacro (robot description, xacro)
@@ -14,5 +14,5 @@
                 <origin rpy="0 0 ${pi/2}" xyz="0 0 ${frame_ground_clearance}"/>
                 <geometry>
-                    <mesh filename="package://robotont_description/meshes/gen2_1/frame_module.STL"/>
+                    <mesh filename="file://$(find robotont_description)/meshes/gen2_1/frame_module.STL"/>
                 </geometry>
                 <material name="base_material">
@@ -22,7 +22,7 @@
             <collision>
                 <geometry>
-                    <mesh filename="package://robotont_description/meshes/shared/collision_body.STL"/>
+                    <mesh filename="file://$(find robotont_description)/meshes/shared/collision_body.STL"/>
                 </geometry>
-                <origin rpy="${pi/2} 0 ${pi/2}"/>
+                <origin rpy="${pi/2} 0 ${pi/2}" xyz="-0.01 0 ${frame_ground_clearance + 0.035}"/>
             </collision>
             <inertial>
@@ -47,5 +47,5 @@
             <visual>
                 <geometry>
-                    <mesh filename="package://robotont_description/meshes/gen3/e_stop_button.STL"/>
+                    <mesh filename="file://$(find robotont_description)/meshes/gen3/e_stop_button.STL"/>
                 </geometry>
                 <material name="e_button_material">
@@ -67,5 +67,5 @@
             <visual>
                 <geometry>
-                    <mesh filename="package://robotont_description/meshes/gen3/power_button.STL"/>
+                    <mesh filename="file://$(find robotont_description)/meshes/gen3/power_button.STL"/>
                 </geometry>
                 <material name="power_button_material">

File: urdf/gen2_1/motor.urdf.xacro (robot description, xacro)
@@ -21,5 +21,5 @@
             <visual>
                 <geometry>
-                    <mesh filename="package://robotont_description/meshes/gen2_1/motor_module.STL"/>
+                    <mesh filename="file://$(find robotont_description)/meshes/gen2_1/motor_module.STL"/>
                 </geometry>
                 <material name="motor_mount_${name}_material">
@@ -40,5 +40,5 @@
             <visual>
                 <geometry>
-                    <mesh filename="package://robotont_description/meshes/gen2_1/motor.STL"/>
+                    <mesh filename="file://$(find robotont_description)/meshes/gen2_1/motor.STL"/>
                 </geometry>
                 <material name="motor_${name}_material">

File: urdf/gen3/base.urdf.xacro (robot description, xacro)
@@ -19,5 +19,5 @@
                 <origin rpy="0 0 ${pi/2}" xyz="0 0 ${frame_elevation}"/>
                 <geometry>
-                    <mesh filename="package://robotont_description/meshes/gen3/frame_module.STL"/>
+                    <mesh filename="file://$(find robotont_description)/meshes/gen3/frame_module.STL"/>
                 </geometry>
                 <material name="base_material">
@@ -27,5 +27,5 @@
             <collision>
                 <geometry>
-                    <mesh filename="package://robotont_description/meshes/shared/collision_body.STL"/>
+                    <mesh filename="file://$(find robotont_description)/meshes/shared/collision_body.STL"/>
                 </geometry>
                 <origin rpy="${pi/2} 0 ${pi/2}" xyz="0 0 ${frame_elevation}"/>
@@ -53,5 +53,5 @@
                 <origin rpy="0 0 ${pi/2}" xyz="0 0 0"/>
                 <geometry>
-                    <mesh filename="package://robotont_description/meshes/gen3/PCB.STL"/>
+                    <mesh filename="file://$(find robotont_description)/meshes/gen3/PCB.STL"/>
                 </geometry>
                 <material name="pcb_material">
@@ -69,5 +69,5 @@
             <visual>
                 <geometry>
-                    <mesh filename="package://robotont_description/meshes/gen3/e_stop_button.STL"/>
+                    <mesh filename="file://$(find robotont_description)/meshes/gen3/e_stop_button.STL"/>
                 </geometry>
                 <material name="e_button_material">
@@ -89,5 +89,5 @@
             <visual>
                 <geometry>
-                    <mesh filename="package://robotont_description/meshes/gen3/power_button.STL"/>
+                    <mesh filename="file://$(find robotont_description)/meshes/gen3/power_button.STL"/>
                 </geometry>
                 <material name="power_button_material">
@@ -109,5 +109,5 @@
             <visual>
                 <geometry>
-                    <mesh filename="package://robotont_description/meshes/gen3/battery_module.STL"/>
+                    <mesh filename="file://$(find robotont_description)/meshes/gen3/battery_module.STL"/>
                 </geometry>
                 <material name="battery_module_material">

File: urdf/gen3/motor.urdf.xacro (robot description, xacro)
@@ -9,5 +9,5 @@
             <visual>
                 <geometry>
-                    <mesh filename="package://robotont_description/meshes/gen3/motor_module.STL"/>
+                    <mesh filename="file://$(find robotont_description)/meshes/gen3/motor_module.STL"/>
                 </geometry>
                 <material name="motor_${name}_material">

File: urdf/shared/rim.urdf.xacro (robot description, xacro)
@@ -11,5 +11,5 @@
             <visual>
                 <geometry>
-                    <mesh filename="package://robotont_description/meshes/shared/rim.STL"/>
+                    <mesh filename="file://$(find robotont_description)/meshes/shared/rim.STL"/>
                 </geometry>
                 <material name="rim_${name}_material">
@@ -43,4 +43,5 @@
                 rpy="${pi/2} 0 ${angle + pi + z_rotation_offset}"
             />
+            <dynamics damping="0.1"/>
         </joint>
         <!-- Front rollers -->

File: urdf/shared/roller.urdf.xacro (robot description, xacro)
@@ -17,5 +17,5 @@
             <visual>
                 <geometry>
-                    <mesh scale="0.001 0.001 0.001" filename="package://robotont_description/meshes/shared/roller.STL"/>
+                    <mesh scale="0.001 0.001 0.001" filename="file://$(find robotont_description)/meshes/shared/roller.STL"/>
                 </geometry>
                 <material name="roller_material">
