Commit message: loading meshes using the package substitute to make it work also for distributed ros

File: urdf/gen2_1/base.urdf.xacro (robot description, xacro)
@@ -14,5 +14,5 @@
                 <origin rpy="0 0 ${pi/2}" xyz="0 0 ${frame_ground_clearance}"/>
                 <geometry>
-                    <mesh filename="file://$(find robotont_description)/meshes/gen2_1/frame_module.STL"/>
+                    <mesh filename="package://robotont_description/meshes/gen2_1/frame_module.STL"/>
                 </geometry>
                 <material name="base_material">
@@ -22,5 +22,5 @@
             <collision>
                 <geometry>
-                    <mesh filename="file://$(find robotont_description)/meshes/shared/collision_body.STL"/>
+                    <mesh filename="package://robotont_description/meshes/shared/collision_body.STL"/>
                 </geometry>
                 <origin rpy="${pi/2} 0 ${pi/2}" xyz="-0.01 0 ${frame_ground_clearance + 0.035}"/>
@@ -47,5 +47,5 @@
             <visual>
                 <geometry>
-                    <mesh filename="file://$(find robotont_description)/meshes/gen3/e_stop_button.STL"/>
+                    <mesh filename="package://robotont_description/meshes/gen3/e_stop_button.STL"/>
                 </geometry>
                 <material name="e_button_material">
@@ -67,5 +67,5 @@
             <visual>
                 <geometry>
-                    <mesh filename="file://$(find robotont_description)/meshes/gen3/power_button.STL"/>
+                    <mesh filename="package://robotont_description/meshes/gen3/power_button.STL"/>
                 </geometry>
                 <material name="power_button_material">

File: urdf/gen2_1/motor.urdf.xacro (robot description, xacro)
@@ -21,5 +21,5 @@
             <visual>
                 <geometry>
-                    <mesh filename="file://$(find robotont_description)/meshes/gen2_1/motor_module.STL"/>
+                    <mesh filename="package://robotont_description/meshes/gen2_1/motor_module.STL"/>
                 </geometry>
                 <material name="motor_mount_${name}_material">
@@ -40,5 +40,5 @@
             <visual>
                 <geometry>
-                    <mesh filename="file://$(find robotont_description)/meshes/gen2_1/motor.STL"/>
+                    <mesh filename="package://robotont_description/meshes/gen2_1/motor.STL"/>
                 </geometry>
                 <material name="motor_${name}_material">

File: urdf/gen3/base.urdf.xacro (robot description, xacro)
@@ -20,5 +20,5 @@
                 <origin rpy="0 0 ${pi/2}" xyz="0 0 ${frame_elevation}"/>
                 <geometry>
-                    <mesh filename="file://$(find robotont_description)/meshes/gen3/frame_module_pla.STL"/>
+                    <mesh filename="package://robotont_description/meshes/gen3/frame_module_pla.STL"/>
                 </geometry>
                 <material name="base_material">
@@ -28,5 +28,5 @@
             <collision>
                 <geometry>
-                    <mesh filename="file://$(find robotont_description)/meshes/shared/collision_body.STL"/>
+                    <mesh filename="package://robotont_description/meshes/shared/collision_body.STL"/>
                 </geometry>
                 <origin rpy="${pi/2} 0 ${pi/2}" xyz="0 0 ${frame_elevation}"/>
@@ -53,5 +53,5 @@
                 <origin rpy="0 0 ${pi/2}" xyz="0 0 ${frame_elevation}"/>
                 <geometry>
-                    <mesh filename="file://$(find robotont_description)/meshes/gen3/frame_module_spacers.STL"/>
+                    <mesh filename="package://robotont_description/meshes/gen3/frame_module_spacers.STL"/>
                 </geometry>
                 <material name="spacers_material">
@@ -70,5 +70,5 @@
                 <origin rpy="0 0 ${pi/2}" xyz="0 0 0"/>
                 <geometry>
-                    <mesh filename="file://$(find robotont_description)/meshes/gen3/PCB.STL"/>
+                    <mesh filename="package://robotont_description/meshes/gen3/PCB.STL"/>
                 </geometry>
                 <material name="pcb_material">
@@ -86,5 +86,5 @@
             <visual>
                 <geometry>
-                    <mesh filename="file://$(find robotont_description)/meshes/gen3/e_stop_button.STL"/>
+                    <mesh filename="package://robotont_description/meshes/gen3/e_stop_button.STL"/>
                 </geometry>
                 <material name="e_button_material">
@@ -106,5 +106,5 @@
             <visual>
                 <geometry>
-                    <mesh filename="file://$(find robotont_description)/meshes/gen3/power_button.STL"/>
+                    <mesh filename="package://robotont_description/meshes/gen3/power_button.STL"/>
                 </geometry>
                 <material name="power_button_material">
@@ -126,5 +126,5 @@
             <visual>
                 <geometry>
-                    <mesh filename="file://$(find robotont_description)/meshes/gen3/encoder_button.STL"/>
+                    <mesh filename="package://robotont_description/meshes/gen3/encoder_button.STL"/>
                 </geometry>
                 <material name="encoder_button_material">
@@ -146,5 +146,5 @@
             <visual>
                 <geometry>
-                    <mesh filename="file://$(find robotont_description)/meshes/gen3/battery_module.STL"/>
+                    <mesh filename="package://robotont_description/meshes/gen3/battery_module.STL"/>
                 </geometry>
                 <material name="battery_module_material">
@@ -166,5 +166,5 @@
             <visual>
                 <geometry>
-                    <mesh filename="file://$(find robotont_description)/meshes/gen3/ssd1306.STL"/>
+                    <mesh filename="package://robotont_description/meshes/gen3/ssd1306.STL"/>
                 </geometry>
                 <material name="screen_module_material">

File: urdf/gen3/motor.urdf.xacro (robot description, xacro)
@@ -22,5 +22,5 @@
             <visual>
                 <geometry>
-                    <mesh filename="file://$(find robotont_description)/meshes/gen3/motor_module2.STL"/>
+                    <mesh filename="package://robotont_description/meshes/gen3/motor_module2.STL"/>
                 </geometry>
                 <material name="motor_${name}_material">

File: urdf/shared/rim.urdf.xacro (robot description, xacro)
@@ -21,5 +21,5 @@
             <visual>
                 <geometry>
-                    <mesh filename="file://$(find robotont_description)/meshes/shared/2.75rim.STL"/>
+                    <mesh filename="package://robotont_description/meshes/shared/2.75rim.STL"/>
                 </geometry>
                 <material name="rim_${name}_material">

File: urdf/shared/roller.urdf.xacro (robot description, xacro)
@@ -17,5 +17,5 @@
             <visual>
                 <geometry>
-                    <mesh scale="0.001 0.001 0.001" filename="file://$(find robotont_description)/meshes/shared/2.75roller.STL"/>
+                    <mesh scale="0.001 0.001 0.001" filename="package://robotont_description/meshes/shared/2.75roller.STL"/>
                 </geometry>
                 <material name="roller_material">
