Commit message: robotont-description - Update gen3 model, move wheel center to correct position

File: urdf/gen3/motor.urdf.xacro (robot description, xacro)
@@ -3,7 +3,20 @@
     xmlns:xacro="http://ros.org/wiki/xacro">
     <xacro:property name="length" value="0.0725"/>
-    <xacro:macro name="motor_macro" params="name color angle z_rotation_offset wheel_center_height wheel_length frame_ground_clearance frame_thickness distance gap prefix">
+    <xacro:macro name="motor_macro" params="
+        name
+        color
+        angle
+        z_rotation:=0
+        position_offset:=1
+        wheel_center_offset
+        wheel_center_height
+        wheel_length
+        frame_ground_clearance
+        frame_thickness
+        distance
+        prefix
+    ">
         <xacro:property name="ground_clearance" value="${1.5 * wheel_center_height + frame_ground_clearance + frame_thickness}"/>
-        <xacro:property name="distance_from_center" value="${distance + (wheel_length / 2) + (length / 2) + gap}"/>
+        <xacro:property name="distance_from_center" value="${distance + (wheel_length / 2) + ((length * position_offset) / 2)}"/>
         <link name="${prefix}motor_${name}_link">
             <visual>
@@ -21,6 +34,6 @@
             <axis xyz="0 0 1"/>
             <origin
-                xyz="${distance_from_center * sin(angle)} ${-distance_from_center * cos(angle)} ${ground_clearance}"
-                rpy="${pi/2} 0 ${angle + pi + z_rotation_offset}"
+                xyz="${distance_from_center * sin(angle) + wheel_center_offset} ${-distance_from_center * cos(angle)} ${ground_clearance}"
+                rpy="${pi/2} 0 ${angle + pi + z_rotation}"
             />
         </joint>

File: urdf/gen3/robotont.urdf.xacro (robot description, xacro)
@@ -6,6 +6,6 @@
     <xacro:arg name="prefix" default=""/>
     <xacro:property name="prefix" value="$(arg prefix)"/>
-    <xacro:property name="wheel_distance_back" value="0.14"/>
-    <xacro:property name="wheel_distance_front" value="0.16"/>
+    <xacro:property name="wheel_distance" value="0.151"/>
+    <xacro:property name="wheel_center_offset" value="0.014"/>
     <xacro:property name="wheel_center_height" value="0.021"/>
     <xacro:property name="roller_color" value="0.61 0.55 0.49 1.0"/>
@@ -38,11 +38,10 @@
         color="${rim_color}"
         angle="${-3 * pi / 2}"
-        z_rotation_offset="0"
         wheel_center_height="${wheel_center_height}"
+        wheel_center_offset="${wheel_center_offset}"
         wheel_length="${wheel_length}"
         frame_ground_clearance="${frame_ground_clearance}"
         frame_thickness="${frame_thickness}"
-        distance="${-wheel_distance_back}"
-        gap="0.0025"
+        distance="${-wheel_distance}"
         prefix="${prefix}"
     />
@@ -50,12 +49,13 @@
         name="right"
         color="${rim_color}"
-        angle="${-143.5 * (pi/180)}"
-        z_rotation_offset="${-wheel_z_rotation_offset}"
+        angle="${5 * pi / 6}"
+        z_rotation="${pi}"
+        position_offset="${-1}"
+        wheel_center_offset="${wheel_center_offset}"
         wheel_center_height="${wheel_center_height}"
-        wheel_length="${wheel_length}"
+        wheel_length="${-wheel_length}"
         frame_ground_clearance="${frame_ground_clearance}"
         frame_thickness="${frame_thickness}"
-        distance="${-wheel_distance_front}"
-        gap="0"
+        distance="${wheel_distance}"
         prefix="${prefix}"
     />
@@ -63,12 +63,11 @@
         name="left"
         color="${rim_color}"
-        angle="${-36.5 * (pi/180)}"
-        z_rotation_offset="${wheel_z_rotation_offset}"
+        angle="${7 * pi / 6}"
+        wheel_center_offset="${wheel_center_offset}"
         wheel_center_height="${wheel_center_height}"
         wheel_length="${wheel_length}"
         frame_ground_clearance="${frame_ground_clearance}"
         frame_thickness="${frame_thickness}"
-        distance="${-wheel_distance_front}"
-        gap="0"
+        distance="${-wheel_distance}"
         prefix="${prefix}"
     />
@@ -78,8 +77,8 @@
         color="${rim_color}"
         roller_color="${roller_color}"
-        angle="${3*pi/2}"
-        wheel_distance="${wheel_distance_back}"
+        angle="${3 * pi / 2}"
+        wheel_distance="${wheel_distance}"
         wheel_center_height="${wheel_center_height}"
-        z_rotation_offset="0"
+        wheel_center_offset="${wheel_center_offset}"
         prefix="${prefix}"
     />
@@ -88,8 +87,8 @@
         color="${rim_color}"
         roller_color="${roller_color}"
-        angle="${145 * (pi/180)}"
-        wheel_distance="${wheel_distance_front}"
+        angle="${5 * pi / 6}"
+        wheel_distance="${wheel_distance}"
         wheel_center_height="${wheel_center_height}"
-        z_rotation_offset="${wheel_z_rotation_offset}"
+        wheel_center_offset="${wheel_center_offset}"
         prefix="${prefix}"
     />
@@ -98,8 +97,8 @@
         color="${rim_color}"
         roller_color="${roller_color}"
-        angle="${35 * (pi/180)}"
-        wheel_distance="${wheel_distance_front}"
+        angle="${7 * pi / 6}"
+        wheel_distance="${-wheel_distance}"
         wheel_center_height="${wheel_center_height}"
-        z_rotation_offset="${-wheel_z_rotation_offset}"
+        wheel_center_offset="${wheel_center_offset}"
         prefix="${prefix}"
     />

File: urdf/shared/rim.urdf.xacro (robot description, xacro)
@@ -7,5 +7,14 @@
     <xacro:property name="roller_init_angle" value="0" />
     <xacro:property name="wheel_height_offset" value="${wheel_center_height / 2}"/>
-    <xacro:macro name="rim_macro" params="name color roller_color angle wheel_distance wheel_center_height z_rotation_offset prefix">
+    <xacro:macro name="rim_macro" params="
+        name
+        color
+        roller_color
+        angle
+        wheel_distance
+        wheel_center_height
+        wheel_center_offset
+        prefix
+    ">
         <link name="${prefix}rim_${name}_link">
             <visual>
@@ -40,6 +49,6 @@
             <axis xyz="0 0 1"/>
             <origin
-                xyz="${wheel_distance * sin(angle)} ${ -wheel_distance * cos(angle)} ${wheel_center_height + wheel_height_offset}"
-                rpy="${pi/2} 0 ${angle + pi + z_rotation_offset}"
+                xyz="${wheel_center_offset + (wheel_distance * sin(angle))} ${ -wheel_distance * cos(angle)} ${wheel_center_height + wheel_height_offset}"
+                rpy="${pi/2} 0 ${angle + pi}"
             />
             <dynamics damping="0.1"/>
