Commit message: metallic color for spacers and new wheels

File: urdf/gen3/base.urdf.xacro (robot description, xacro)
@@ -1,8 +1,9 @@
 <?xml version="1.0"?>
 <robot xmlns:xacro="http://ros.org/wiki/xacro">
-    <xacro:property name="pcb_offset" value="0.044"/>
+    <xacro:property name="pcb_offset" value="0.0444"/>
     <xacro:property name="e_button_offset" value="0.0035"/>
     <xacro:macro name="base_macro" params="
         color
+        spacers_color
         pcb_color
         e_button_color
@@ -13,11 +14,11 @@
         prefix
     ">
-        <xacro:property name="frame_elevation" value="${frame_height / 2 + frame_ground_clearance}"/>
+        <xacro:property name="frame_elevation" value="${frame_height / 2 + frame_ground_clearance+0.004}"/>
         <!-- Frame -->
         <link name="${prefix}base_link">
             <visual>
-                <origin rpy="0 0 ${pi/2}" xyz="0 0 ${frame_elevation}"/>
+                <origin rpy="0 0 ${pi/2}" xyz="0.0042 0 ${frame_elevation}"/>
                 <geometry>
-                    <mesh filename="file://$(find robotont_description)/meshes/gen3/frame_module.STL"/>
+                    <mesh scale="0.001 0.001 0.001" filename="file://$(find robotont_description)/meshes/gen3/frame_module_pla.STL"/>
                 </geometry>
                 <material name="base_material">
@@ -46,5 +47,21 @@
             <parent link="${prefix}base_footprint"/>
             <child link="${prefix}base_link"/>
-            <origin xyz="0 0 ${frame_elevation}" rpy="0 0 0"/>
+            <origin xyz="0 0 0" rpy="0 0 ${frame_elevation}"/>
+        </joint>
+        <link name="${prefix}base_link_spacers">
+            <visual>
+                <origin rpy="0 0 ${pi/2}" xyz="0.0042 0 ${frame_elevation}"/>
+                <geometry>
+                    <mesh scale="0.001 0.001 0.001" filename="file://$(find robotont_description)/meshes/gen3/frame_module_spacers.STL"/>
+                </geometry>
+                <material name="spacers_material">
+                    <color rgba="${spacers_color}"/>
+                </material>
+            </visual>
+        </link>
+        <joint name="${prefix}base_joint_spacers" type="fixed">
+            <parent link="${prefix}base_footprint"/>
+            <child link="${prefix}base_link_spacers"/>
+            <origin xyz="0 0 0" rpy="0 0 ${frame_elevation}"/>
         </joint>
         <!-- PCB -->

File: urdf/gen3/robotont.urdf.xacro (robot description, xacro)
@@ -14,4 +14,5 @@
     <xacro:property name="wheel_length" value="${0.0225}"/>
     <xacro:property name="frame_height" value="0.065"/>
+    <xacro:property name="spacers_color" value="0.8 0.8 0.8 1.0"/>
     <xacro:property name="frame_ground_clearance" value="0.014"/>
     <xacro:property name="frame_thickness" value="0.000025"/>
@@ -25,4 +26,5 @@
     <xacro:base_macro
         color="${base_color}"
+        spacers_color="${spacers_color}"
         pcb_color="${pcb_color}"
         e_button_color="${e_button_color}"

File: urdf/shared/rim.urdf.xacro (robot description, xacro)
@@ -3,5 +3,5 @@
     xmlns:xacro="http://ros.org/wiki/xacro">
     <xacro:include filename="$(find robotont_description)/urdf/shared/roller.urdf.xacro"/>
-    <xacro:property name="roller_radial_dist" value="0.0275" />
+    <xacro:property name="roller_radial_dist" value="0.0295" />
     <xacro:property name="roller_z_distance" value="0.008" />
     <xacro:property name="roller_init_angle" value="0" />
@@ -21,5 +21,5 @@
             <visual>
                 <geometry>
-                    <mesh filename="file://$(find robotont_description)/meshes/shared/rim.STL"/>
+                    <mesh filename="file://$(find robotont_description)/meshes/shared/2.75rim.STL"/>
                 </geometry>
                 <material name="rim_${name}_material">
@@ -126,4 +126,24 @@
             prefix="${prefix}"
         />
+        <xacro:roller_macro
+            parent="${name}"
+            color="${roller_color}"
+            radial_dist="${roller_radial_dist}"
+            z_distance="${roller_z_distance}"
+            z_distance_reflect="-1"
+            init_angle="${roller_init_angle}"
+            no_of_roller="7"
+            prefix="${prefix}"
+        />
+        <xacro:roller_macro
+            parent="${name}"
+            color="${roller_color}"
+            radial_dist="${roller_radial_dist}"
+            z_distance="${roller_z_distance}"
+            z_distance_reflect="-1"
+            init_angle="${roller_init_angle}"
+            no_of_roller="8"
+            prefix="${prefix}"
+        />
         <!-- Back rollers -->
         <xacro:roller_macro
@@ -195,4 +215,24 @@
             init_angle="${roller_init_angle}"
             no_of_roller="6"
+            prefix="${prefix}"
+        />
+        <xacro:roller_macro
+            parent="${name}"
+            color="${roller_color}"
+            radial_dist="${roller_radial_dist}"
+            z_distance="${roller_z_distance}"
+            z_distance_reflect="1"
+            init_angle="${roller_init_angle}"
+            no_of_roller="7"
+            prefix="${prefix}"
+        />
+        <xacro:roller_macro
+            parent="${name}"
+            color="${roller_color}"
+            radial_dist="${roller_radial_dist}"
+            z_distance="${roller_z_distance}"
+            z_distance_reflect="1"
+            init_angle="${roller_init_angle}"
+            no_of_roller="8"
             prefix="${prefix}"
         />

File: urdf/shared/roller.urdf.xacro (robot description, xacro)
@@ -17,5 +17,5 @@
             <visual>
                 <geometry>
-                    <mesh scale="0.001 0.001 0.001" filename="file://$(find robotont_description)/meshes/shared/roller.STL"/>
+                    <mesh scale="0.001 0.001 0.001" filename="file://$(find robotont_description)/meshes/shared/2.75roller.STL"/>
                 </geometry>
                 <material name="roller_material">
@@ -36,6 +36,6 @@
             <child link="${prefix}roller_${name}_rim_${parent}_link"/>
             <origin
-				xyz="${radial_dist*sin(-1*z_distance_reflect*(init_angle+offset+no_of_roller*2*pi/7))} ${-radial_dist*cos(-1*z_distance_reflect*(init_angle+offset+no_of_roller*2*pi/7))} ${z_distance*z_distance_reflect}"
-				rpy="0 0 ${-1*z_distance_reflect*(init_angle+no_of_roller*2*pi/7)}"
+				xyz="${radial_dist*sin(-1*z_distance_reflect*(init_angle+offset+no_of_roller*2*pi/9))} ${-radial_dist*cos(-1*z_distance_reflect*(init_angle+offset+no_of_roller*2*pi/9))} ${z_distance*z_distance_reflect}"
+				rpy="0 0 ${-1*z_distance_reflect*(init_angle+no_of_roller*2*pi/9)}"
 			/>
         </joint>

Commit message: new wheel to motor adapter, encoder button, launch parameters color

File: urdf/gen3/base.urdf.xacro (robot description, xacro)
@@ -1,5 +1,5 @@
 <?xml version="1.0"?>
 <robot xmlns:xacro="http://ros.org/wiki/xacro">
-    <xacro:property name="pcb_offset" value="0.0444"/>
+    <xacro:property name="pcb_offset" value="0.044"/>
     <xacro:property name="e_button_offset" value="0.0035"/>
     <xacro:macro name="base_macro" params="
@@ -14,9 +14,9 @@
         prefix
     ">
-        <xacro:property name="frame_elevation" value="${frame_height / 2 + frame_ground_clearance+0.004}"/>
+        <xacro:property name="frame_elevation" value="${frame_height / 2 + frame_ground_clearance}"/>
         <!-- Frame -->
         <link name="${prefix}base_link">
             <visual>
-                <origin rpy="0 0 ${pi/2}" xyz="0.0042 0 ${frame_elevation}"/>
+                <origin rpy="0 0 ${pi/2}" xyz="0 0 ${frame_elevation}"/>
                 <geometry>
                     <mesh scale="0.001 0.001 0.001" filename="file://$(find robotont_description)/meshes/gen3/frame_module_pla.STL"/>
@@ -51,5 +51,5 @@
         <link name="${prefix}base_link_spacers">
             <visual>
-                <origin rpy="0 0 ${pi/2}" xyz="0.0042 0 ${frame_elevation}"/>
+                <origin rpy="0 0 ${pi/2}" xyz="0 0 ${frame_elevation}"/>
                 <geometry>
                     <mesh scale="0.001 0.001 0.001" filename="file://$(find robotont_description)/meshes/gen3/frame_module_spacers.STL"/>
@@ -122,4 +122,24 @@
             />
         </joint>
+        <!-- Encoder button -->
+        <link name="${prefix}encoder_button_link">
+            <visual>
+                <geometry>
+                    <mesh filename="file://$(find robotont_description)/meshes/gen3/encoder_button.STL"/>
+                </geometry>
+                <material name="encoder_button_material">
+                    <color rgba="${power_button_color}"/>
+                </material>
+            </visual>
+        </link>
+        <joint name="encoder_button_joint" type="fixed">
+            <parent link="${prefix}base_link"/>
+            <child link="${prefix}encoder_button_link"/>
+            <axis xyz="0 0 1"/>
+            <origin
+                xyz="-0.07 0.12 ${frame_ground_clearance + frame_height - 0.007}"
+                rpy="0 0 0"
+            />
+        </joint>
         <!-- Battery module -->
         <link name="${prefix}battery_module_link">

File: urdf/gen3/motor.urdf.xacro (robot description, xacro)
@@ -22,5 +22,5 @@
             <visual>
                 <geometry>
-                    <mesh filename="file://$(find robotont_description)/meshes/gen3/motor_module.STL"/>
+                    <mesh filename="file://$(find robotont_description)/meshes/gen3/motor_module2.STL"/>
                 </geometry>
                 <material name="motor_${name}_material">

File: urdf/gen3/robotont.urdf.xacro (robot description, xacro)
@@ -6,4 +6,5 @@
     <xacro:arg name="prefix" default=""/>
     <xacro:property name="prefix" value="$(arg prefix)"/>
+    <xacro:property name="primary_color" value="$(arg main_color)"/>
     <xacro:property name="wheel_distance" value="0.151"/>
     <xacro:property name="wheel_center_offset" value="0.014"/>
@@ -25,5 +26,5 @@
     <!-- Frame module -->
     <xacro:base_macro
-        color="${base_color}"
+        color="${primary_color}"
         spacers_color="${spacers_color}"
         pcb_color="${pcb_color}"

Commit message: OLED screen

File: urdf/gen3/base.urdf.xacro (robot description, xacro)
@@ -162,4 +162,24 @@
             />
         </joint>
+        <!-- OLED module -->
+        <link name="${prefix}screen_module_link">
+            <visual>
+                <geometry>
+                    <mesh filename="file://$(find robotont_description)/meshes/gen3/ssd1306.STL"/>
+                </geometry>
+                <material name="screen_module_material">
+                    <color rgba="${battery_module_color}"/>
+                </material>
+            </visual>
+        </link>
+        <joint name="screen_module_joint" type="fixed">
+            <parent link="${prefix}base_link"/>
+            <child link="${prefix}screen_module_link"/>
+            <axis xyz="0 0 1"/>
+            <origin
+                xyz="-0.0325 0.1185 ${frame_ground_clearance + frame_height-0.0015}"
+                rpy="0 0 0"
+            />
+        </joint>
     </xacro:macro>
 </robot>

Commit message: fix scale

File: urdf/gen3/base.urdf.xacro (robot description, xacro)
@@ -20,5 +20,5 @@
                 <origin rpy="0 0 ${pi/2}" xyz="0 0 ${frame_elevation}"/>
                 <geometry>
-                    <mesh scale="0.001 0.001 0.001" filename="file://$(find robotont_description)/meshes/gen3/frame_module_pla.STL"/>
+                    <mesh filename="file://$(find robotont_description)/meshes/gen3/frame_module_pla.STL"/>
                 </geometry>
                 <material name="base_material">
@@ -53,5 +53,5 @@
                 <origin rpy="0 0 ${pi/2}" xyz="0 0 ${frame_elevation}"/>
                 <geometry>
-                    <mesh scale="0.001 0.001 0.001" filename="file://$(find robotont_description)/meshes/gen3/frame_module_spacers.STL"/>
+                    <mesh filename="file://$(find robotont_description)/meshes/gen3/frame_module_spacers.STL"/>
                 </geometry>
                 <material name="spacers_material">

Commit message: typo

File: urdf/gen3/base.urdf.xacro (robot description, xacro)
@@ -47,5 +47,5 @@
             <parent link="${prefix}base_footprint"/>
             <child link="${prefix}base_link"/>
-            <origin xyz="0 0 0" rpy="0 0 ${frame_elevation}"/>
+            <origin xyz="0 0 0" rpy="0 0 0"/>
         </joint>
         <link name="${prefix}base_link_spacers">
